File: hw/ethercat.kicad_sch (KiCad schematic)
At the start: 9 parts, among them J1 RJ45_LED_Shielded, U2 M24C01-RMN

Commit message: Update ethercat circuit
Parts:
- removed J1: RJ45_LED_Shielded, symbol Connector:RJ45_LED_Shielded
- added J1, J2: RJ45_Abracon_ARJC07-111071A, symbol ethercat:RJ45_Abracon_ARJC07-111071A
- added R1, R2: 49.9, symbol Device:R
Connections:
- net TXNA: now reaches U1.52 (TXNA)
- net TXNA: now also R2.2
- net TXPA: now reaches U1.53 (TXPA)
- net TXPA: now also R1.2
- net RXNA: now reaches U1.54 (RXNA)
- net RXPA: now reaches U1.55 (RXPA)
Other:
- moved on the sheet: U2
